File: Electrical Design/macropad/macropad.kicad_pcb (KiCad board)
At the start: 2 copper layers, 100 x 116 mm, 116 parts, among them J1 SM04B-SRSS-TB, SW1 keyswitch, SW10 keyswitch, SW11 keyswitch, SW12 keyswitch, SW13 keyswitch, SW14 keyswitch, SW15 keyswitch, SW16 keyswitch, SW17 keyswitch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

Commit message: Centered XIAO RP2040 and moved around some footprints to accommodate its new placement.
Parts:
- moved D21 20.9 mm to (75.1, 52.3)
- moved U1 8.43 mm to (114.9, 55.8)
- moved R1 5.64 mm to (71.6, 74.0)
- moved U3 3.96 mm to (96.4, 60.5)
- moved C1 3.65 mm to (63.8, 77.6)
- moved U2 3.65 mm to (70.0, 79.4)
Routing:
- net Net-(D21-A): track 7.95 -> 24.0 mm
- net /SDA: track 98.7 -> 110.8 mm
- net /ROW6: track 85.8 -> 97.0 mm
- net /LED: track 41.8 -> 52.0 mm
- net /ENC2_B: track 19.1 -> 27.7 mm
- net /SLIDE: track 67.4 -> 59.1 mm
- net /ENC2_A: track 15.6 -> 23.8 mm
- net +3V3: track 133.2 -> 141.0 mm
- net /SCL: track 99.8 -> 107.3 mm
- net /ENC_A: track 66.4 -> 61.2 mm
- net /ROW5: track 139.9 -> 135.3 mm
- net /ROW3: track 112.5 -> 108.1 mm
- net /ROW4: track 128.7 -> 124.5 mm
- net /ENC_B: track 41.5 -> 37.8 mm
- net /COL4: track 179.1 -> 175.5 mm
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Other:
- outline, holes or cut-outs redrawn
